File: kicad/mc68000board/retrp_mc68000p10/retrp_mc68000p10.kicad_sch (KiCad schematic)
At the start: 13 parts, among them J1 Screw_Terminal_01x02, J2 Conn_02x32_Odd_Even, U1 68000D

Commit message: #1 now with rendered image
Parts:
- added D1: Green, Diode_SMD:D_0805_2012Metric, symbol Device:LED
- added R1: 300, Resistor_SMD:R_0805_2012Metric, symbol Device:R
Connections:
- net GND: now also D1.1 (K)
- net VCC: now also R1.1
- new net: D1.2 (A), R1.2
Changed lines of the file:
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@@
+    (stroke (width 0) (type default))
+  )
+  (wire (pts (xy 68.58 22.86) (xy 71.12 22.86))
     (stroke (width 0) (type default))
   )
@@
     )
   )
-  (global_label "nVPA" (shape input) (at 199.39 138.43 180) (fields_autoplaced)
-    (effects (font (size 1.27 1.27)) (justify right))
-    (property "Intersheetrefs" "${INTERSHEET_REFS}" (at 191.888 138.43 0)
+  (global_label "nVPA" (shape input) (at 173.99 123.19 180) (fields_autoplaced)
+    (effects (font (size 1.27 1.27)) (justify right))
+    (property "Intersheetrefs" "${INTERSHEET_REFS}" (at 166.488 123.19 0)
       (effects (font (size 1.27 1.27)) (justify right) hide)
     )
@@
     (property "Intersheetrefs" "${INTERSHEET_REFS}" (at 75.6528 62.23 0)
       (effects (font (size 1.27 1.27)) (justify right) hide)
+    )
+  )
+  (symbol (lib_id "Device:R") (at 64.77 22.86 90) (unit 1)
+    (in_bom yes) (on_board yes) (dnp no) (fields_autoplaced)
+    (property "Reference" "R1" (at 64.77 18.8341 90)
+      (effects (font (size 1.27 1.27)))
+    )
+    (property "Value" "300" (at 64.77 20.7551 90)
+      (effects (font (size 1.27 1.27)))
+    )
+    (property "Footprint" "Resistor_SMD:R_0805_2012Metric" (at 64.77 24.638 90)
+      (effects (font (size 1.27 1.27)) hide)
+    )
+    (property "Datasheet" "~" (at 64.77 22.86 0)
+      (effects (font (size 1.27 1.27)) hide)
+    )
+    (pin "1")
+    (pin "2")
+    (instances
+      (project "retrp_mc68000p10"
+        (path "/af8b6169-2e4f-4ffe-8e63-977c4018eb1b"
+          (reference "R1") (unit 1)
+        )
+      )
     )
   )
@@
     )
   )
+  (symbol (lib_id "power:GND") (at 71.12 30.48 0) (unit 1)
+    (in_bom yes) (on_board yes) (dnp no)
+    (property "Reference" "#PWR010" (at 71.12 36.83 0)
+      (effects (font (size 1.27 1.27)) hide)
+    )
+    (property "Value" "GND" (at 73.66 34.29 0)
+      (effects (font (size 1.27 1.27)))
+    )
+    (property "Footprint" "" (at 71.12 30.48 0)
+      (effects (font (size 1.27 1.27)) hide)
+    )
+    (property "Datasheet" "" (at 71.12 30.48 0)
+      (effects (font (size 1.27 1.27)) hide)
+    )
+    (pin "1")
+    (instances
+      (project "retrp_mc68000p10"
+        (path "/af8b6169-2e4f-4ffe-8e63-977c4018eb1b"
+          (reference "#PWR010") (unit 1)
+        )
+      )
+    )
+  )
   (symbol (lib_id "CPU_NXP_68000:68000D") (at 109.22 110.49 0) (unit 1)
     (in_bom yes) (on_board yes) (dnp no) (fields_autoplaced)
@@
     )
   )
+  (symbol (lib_id "power:VCC") (at 60.96 22.86 90) (unit 1)
+    (in_bom yes) (on_board yes) (dnp no)
+    (property "Reference" "#PWR09" (at 64.77 22.86 0)
+      (effects (font (size 1.27 1.27)) hide)
+    )
+    (property "Value" "VCC" (at 57.15 20.32 0)
+      (effects (font (size 1.27 1.27)))
+    )
+    (property "Footprint" "" (at 60.96 22.86 0)
+      (effects (font (size 1.27 1.27)) hide)
+    )
+    (property "Datasheet" "" (at 60.96 22.86 0)
+      (effects (font (size 1.27 1.27)) hide)
+    )
+    (pin "1")
+    (instances
+      (project "retrp_mc68000p10"
+        (path "/af8b6169-2e4f-4ffe-8e63-977c4018eb1b"
+          (reference "#PWR09") (unit 1)
+        )
+      )
+    )
+  )
   (symbol (lib_id "power:VCC") (at 233.68 22.86 0) (unit 1)
     (in_bom yes) (on_board yes) (dnp no) (fields_autoplaced)
@@
         )
       )
+    )
+  )
+  (symbol (lib_id "Device:LED") (at 71.12 26.67 90) (unit 1)
+    (in_bom yes) (on_board yes) (dnp no) (fields_autoplaced)
+    (property "Reference" "D1" (at 74.041 27.6138 90)
+      (effects (font (size 1.27 1.27)) (justify right))
+    )
+    (property "Value" "Green" (at 74.041 29.5348 90)
+      (effects (font (size 1.27 1.27)) (justify right))
+    )
+    (property "Footprint" "Diode_SMD:D_0805_2012Metric" (at 71.12 26.67 0)
+      (effects (font (size 1.27 1.27)) hide)
+    )
+    (property "Datasheet" "~" (at 71.12 26.67 0)
+      (effects (font (size 1.27 1.27)) hide)
+    )
+    (pin "1")
+    (pin "2")
+    (instances
+      (project "retrp_mc68000p10"
+        (path "/af8b6169-2e4f-4ffe-8e63-977c4018eb1b"
+          (reference "D1") (unit 1)
+        )
+      )
